Commit message: new arm

File: src/complete_assembly/urdf/complete_assembly.urdf (robot description, URDF)
Before this commit: robot complete_assembly, 13 links, 12 joints
Links:
- removed link gripper_base
- added link base_link
- added link gripper, mass 0.0160520536785178; collision mesh filename=package://complete_assembly/meshes/gripper.STL; visual mesh filename=package://complete_assembly/meshes/gripper.STL
- link elbow: mass 0.089627712115124 -> 0.0896278030340915
- link left_finger: mass 0.0053139252062326 -> 0.00531392171589627
- link right_finger: mass 0.00531391451356127 -> 0.00531392173232632
- link rotating_base: mass 0.118965881840798 -> 0.118965826503535
- link shoulder: mass 0.173985874606989 -> 0.173985862227821
- link wrist: mass 0.0159128075867897 -> 0.0159127959387036
Joints:
- added joint base_link_to_fixed_base: type fixed, parent base_link, child fixed_base, origin xyz=0.0 0.0 0.0 rpy=0.0 0.0 0.0
- joint elbow_joint: axis -1 0 0 -> 0 0 1; limit lower=-1.57 upper=1.57 effort=0 velocity=0 -> lower=-1.57 upper=1.57 effort=1 velocity=1; origin xyz=0 -0.27982 0.010033 rpy=0 0 0 -> xyz=0 -0.28 0 rpy=0 0 -0.77026
- joint gripper_joint: child gripper_base -> gripper; limit lower=-1.57 upper=1.57 effort=0 velocity=0 -> lower=-1.57 upper=1.57 effort=1 velocity=1; origin xyz=0.018288 0.012361 0.02425 rpy=-1.5708 1.1957 -1.2049 -> xyz=-0.020533 0.02425 -0.0081026 rpy=2.1829 0.14928 -1.4667
- joint left_finger_joint: axis 0 -1 0 -> -1 0 0; limit lower=-1.57 upper=1.57 effort=0 velocity=0 -> lower=-1.57 upper=1.57 effort=1 velocity=1; origin xyz=-0.027551 -0.00725 -0.013656 rpy=3.1416 0 0 -> xyz=-0.00725 -0.017383 -0.025365 rpy=3.1416 0 -3.1416
- joint left_gear_joint: axis 0 -1 0 -> -1 0 0; limit lower=-1.57 upper=1.57 effort=0 velocity=0 -> lower=-1.57 upper=1.57 effort=1 velocity=1; origin xyz=-0.041365 -0.009685 -0.0085012 rpy=-3.1416 -0.7769 -0.23367 -> xyz=-0.023 -0.03572 -0.0085012 rpy=-0.68328 0 -1.0357; parent gripper_base -> gripper
- joint left_link_joint: axis 0 -1 0 -> -1 0 0; limit lower=-1.57 upper=1.57 effort=0 velocity=0 -> lower=-1.57 upper=1.57 effort=1 velocity=1; origin xyz=-0.060132 -0.0021342 -0.00049887 rpy=-3.1416 -0.7769 -0.23367 -> xyz=-0.041738 -0.04334 -0.00049887 rpy=-0.68328 0 -1.0357; parent gripper_base -> gripper
- joint right_finger_joint: axis 0 -1 0 -> 1 0 0; limit lower=-1.57 upper=1.57 effort=0 velocity=0 -> lower=-1.57 upper=1.57 effort=1 velocity=1; origin xyz=-0.014777 -0.00725 -0.026967 rpy=3.1416 0 0 -> xyz=-0.00725 -0.028069 -0.012558 rpy=0 0 0
- joint right_gear_joint: axis 0 -1 0 -> -1 0 0; limit lower=-1.57 upper=1.57 effort=0 velocity=0 -> lower=-1.57 upper=1.57 effort=1 velocity=1; origin xyz=-0.041365 -0.009685 0.018398 rpy=-3.1416 -0.7769 -0.23367 -> xyz=-0.023 -0.03572 0.018398 rpy=-0.68328 0 -1.0357; parent gripper_base -> gripper
- joint right_link_joint: axis 0 -1 0 -> -1 0 0; limit lower=-1.57 upper=1.57 effort=0 velocity=0 -> lower=-1.57 upper=1.57 effort=1 velocity=1; origin xyz=-0.060132 -0.0021342 0.0095011 rpy=3.1416 -0.7769 -0.23367 -> xyz=-0.041738 -0.04334 0.0095011 rpy=-0.68328 0 -1.0357; parent gripper_base -> gripper
- joint rotating_base_joint: axis 0 -1 0 -> 0 1 0; limit lower=-3.14 upper=3.14 effort=0 velocity=0 -> lower=-3.14 upper=3.14 effort=1 velocity=1; origin xyz=-0.013782 0.034682 0.0071238 rpy=-1.1076 -0.0065997 -0.003296 -> xyz=-0.013849 0.030652 0.015193 rpy=-1.8219 0.39346 -2.177
- joint shoulder_joint: axis -1 0 0 -> 0 0 1; origin xyz=-0.0079307 0.058 -0.0089693 rpy=0.33715 -0.80764 -3.1416 -> xyz=0 0.06702 -0.011931 rpy=1.5708 -1.154 1.5708
- joint wrist_joint: axis 0 0 0 -> 0 1 0; limit (none) -> lower=-1.57 upper=1.57 effort=1 velocity=1; origin xyz=-0.0085 -0.12804 -0.14317 rpy=-2.4731 -0.23314 -2.857 -> xyz=0.192 0.0053 0.0095 rpy=3.1416 0.96644 1.5708; type fixed -> revolute

File: src/pca9685_arm_robot/urdf/arm_robot_ros2_control_block.urdf (robot description, URDF)
Before this commit: robot arm_robot_pkg, 7 links, 6 joints
Links:
- removed link Elbow_link
- removed link shoulder_link
- removed link wrist_link
- added link elbow, mass 0.0896278030340915; collision mesh filename=package://pca9685_arm_robot/meshes/elbow.STL; visual mesh filename=package://pca9685_arm_robot/meshes/elbow.STL
- added link fixed_base, mass 0.0944551427512308; collision mesh filename=package://pca9685_arm_robot/meshes/fixed_base.STL; visual mesh filename=package://pca9685_arm_robot/meshes/fixed_base.STL
- added link left_finger, mass 0.00531392171589627; collision mesh filename=package://pca9685_arm_robot/meshes/left_finger.STL; visual mesh filename=package://pca9685_arm_robot/meshes/left_finger.STL
- added link left_gear, mass 0.00645515105378561; collision mesh filename=package://pca9685_arm_robot/meshes/left_gear.STL; visual mesh filename=package://pca9685_arm_robot/meshes/left_gear.STL
- added link left_link, mass 0.000819182765433022; collision mesh filename=package://pca9685_arm_robot/meshes/left_link.STL; visual mesh filename=package://pca9685_arm_robot/meshes/left_link.STL
- added link right_finger, mass 0.00531392173232632; collision mesh filename=package://pca9685_arm_robot/meshes/right_finger.STL; visual mesh filename=package://pca9685_arm_robot/meshes/right_finger.STL
- added link right_gear, mass 0.00645515105378562; collision mesh filename=package://pca9685_arm_robot/meshes/right_gear.STL; visual mesh filename=package://pca9685_arm_robot/meshes/right_gear.STL
- added link right_link, mass 0.000819182765433024; collision mesh filename=package://pca9685_arm_robot/meshes/right_link.STL; visual mesh filename=package://pca9685_arm_robot/meshes/right_link.STL
- added link shoulder, mass 0.173985862227821; collision mesh filename=package://pca9685_arm_robot/meshes/shoulder.STL; visual mesh filename=package://pca9685_arm_robot/meshes/shoulder.STL
- added link wrist, mass 0.0159127959387036; collision mesh filename=package://pca9685_arm_robot/meshes/wrist.STL; visual mesh filename=package://pca9685_arm_robot/meshes/wrist.STL
- link base_link: mass 0.14496 -> None; geometry 
- link gripper: mass 0.0404906779655548 -> 0.0160520536785178
- link rotating_base: mass 0.072452 -> 0.118965826503535
Joints:
- removed joint Elbow_link_joint
- removed joint shoulder_link_joint
- removed joint wrist_link_joint
- added joint base_link_to_fixed_base: type fixed, parent base_link, child fixed_base, origin xyz=0.0 0.0 0.0 rpy=0.0 0.0 0.0
- added joint elbow_joint: type revolute, parent shoulder, child elbow, origin xyz=0 -0.28 0 rpy=0 0 -0.77026, axis 0 0 1, limit lower=-1.57 upper=1.57 effort=1 velocity=1
- added joint left_finger_joint: type revolute, parent left_gear, child left_finger, origin xyz=-0.00725 -0.017383 -0.025365 rpy=3.1416 0 -3.1416, axis -1 0 0, limit lower=-1.57 upper=1.57 effort=1 velocity=1, mimic joint=right_gear_joint multiplier=1 offset=0
- added joint left_gear_joint: type revolute, parent gripper, child left_gear, origin xyz=-0.023 -0.03572 -0.0085012 rpy=-0.68328 0 -1.0357, axis -1 0 0, limit lower=-1.57 upper=1.57 effort=1 velocity=1, mimic joint=right_gear_joint multiplier=1 offset=0
- added joint left_link_joint: type revolute, parent gripper, child left_link, origin xyz=-0.041738 -0.04334 -0.00049887 rpy=-0.68328 0 -1.0357, axis -1 0 0, limit lower=-1.57 upper=1.57 effort=1 velocity=1, mimic joint=right_gear_joint multiplier=1 offset=0
- added joint right_finger_joint: type revolute, parent right_gear, child right_finger, origin xyz=-0.00725 -0.028069 -0.012558 rpy=0 0 0, axis 1 0 0, limit lower=-1.57 upper=1.57 effort=1 velocity=1, mimic joint=right_gear_joint multiplier=1 offset=0
- added joint right_gear_joint: type revolute, parent gripper, child right_gear, origin xyz=-0.023 -0.03572 0.018398 rpy=-0.68328 0 -1.0357, axis -1 0 0, limit lower=-1.57 upper=1.57 effort=1 velocity=1
- added joint right_link_joint: type revolute, parent gripper, child right_link, origin xyz=-0.041738 -0.04334 0.0095011 rpy=-0.68328 0 -1.0357, axis -1 0 0, limit lower=-1.57 upper=1.57 effort=1 velocity=1, mimic joint=right_gear_joint multiplier=1 offset=0
- added joint shoulder_joint: type revolute, parent rotating_base, child shoulder, origin xyz=0 0.06702 -0.011931 rpy=1.5708 -1.154 1.5708, axis 0 0 1, limit lower=-1.57 upper=1.57 effort=1 velocity=1
- added joint wrist_joint: type revolute, parent elbow, child wrist, origin xyz=0.192 0.0053 0.0095 rpy=3.1416 0.96644 1.5708, axis 0 1 0, limit lower=-1.57 upper=1.57 effort=1 velocity=1
- joint gripper_joint: axis 1 0 0 -> 0 0 -1; limit lower=-1.57 upper=1.57 effort=5 velocity=0 -> lower=-1.57 upper=1.57 effort=1 velocity=1; origin xyz=0.005 0.043353 0 rpy=-1.9228 -1.5708 1.1777 -> xyz=-0.020533 0.02425 -0.0081026 rpy=2.1829 0.14928 -1.4667; parent wrist_link -> wrist
- joint rotating_base_joint: limit lower=-1.046 upper=1.046 effort=7 velocity=0 -> lower=-3.14 upper=3.14 effort=1 velocity=1; origin xyz=0 0 0.0534 rpy=1.5708 0 1.5083 -> xyz=-0.013849 0.030652 0.015193 rpy=-1.8219 0.39346 -2.177; parent base_link -> fixed_base
